Commit message: 坂道_10per

File: urdf/materials.xacro (robot description, xacro)
@@ -1,4 +1,24 @@
 <?xml version="1.0" ?>
 <robot name="vehicle_4ws" xmlns:xacro="http://www.ros.org/wiki/xacro" >
+<xacro:macro name="box_inertia" params="m x y z">
+	    <inertia ixx="${m*(y*y+z*z)/12}" ixy = "0" ixz = "0"
+	             iyy="${m*(z*z+x*x)/12}" iyz = "0"
+	             izz="${m*(x*x+y*y)/12}" />
+	  </xacro:macro>
+	  <xacro:macro name="cariier_inertia" params="m x y z">
+	    <inertia ixx="${m*(y*y+z*z)/12}" ixy = "0" ixz = "0"
+	             iyy="${m*(z*z+x*x)/12}" iyz = "0"
+	             izz="${m*(x*x+y*y)/12}" />
+	  </xacro:macro>
+	  <xacro:macro name="cylinder_inertia" params="m r h">
+	    <inertia ixx="${m*(3*r*r+h*h)/12}" ixy="0" ixz="0"
+	             iyy="${m*(3*r*r+h*h)/12}" iyz="0"
+	             izz="${m*r*r/2}" />
+	  </xacro:macro>
+	  <xacro:macro name="sphere_inertia" params="m r">
+	    <inertia ixx="${m*r*r/5}" ixy="0" ixz="0"
+	             iyy="${m*r*r/5}" iyz="0"
+	             izz="${m*r*r/5}" />
+	  </xacro:macro>
 <material name="silver_default">
   <color rgba="0.700 0.700 0.700 1.000"/>
