Commit message: 0623

File: urdf/vehicle_4ws_real.xacro (robot description, xacro)
@@ -371,4 +371,5 @@
   <child link="new_wheel_1"/>
   <dynamics damping="${front_wheel_joint_damping}" friction="${front_wheel_joint_friction}"/>
+  <limit effort="500" velocity="500"/>
   <axis xyz="0.0 1.0 -0.0"/>
 </joint>
@@ -378,5 +379,5 @@
   <child link="new_wheel_2"/>
   <dynamics damping="${wheel_joint_damping}" friction="${wheel_joint_friction}"/>
-  <limit effort="100" velocity="100"/>
+  <limit effort="500" velocity="500"/>
   <axis xyz="0.0 1.0 -0.0"/>
 </joint>
@@ -394,4 +395,5 @@
   <child link="new_wheel_3"/>
   <dynamics damping="${front_wheel_joint_damping}" friction="${front_wheel_joint_friction}"/>
+  <limit effort="500" velocity="500"/>
   <axis xyz="0.0 1.0 -0.0"/>
 </joint>
@@ -401,5 +403,5 @@
   <child link="new_wheel_4"/>
   <dynamics damping="${wheel_joint_damping}" friction="${wheel_joint_friction}"/>
-  <limit effort="100" velocity="100"/>
+  <limit effort="500" velocity="500"/>
   <axis xyz="0.0 1.0 -0.0"/>
 </joint>

Commit message: 暫定

File: urdf/vehicle_4ws_real.xacro (robot description, xacro)
@@ -40,5 +40,5 @@
 <link name="body_link">
   <inertial>
-    <origin xyz="0.001411408730126027 0.05751189617802702 0.2" rpy="0 0 0"/>
+    <origin xyz="0.001411408730126027 0.05751189617802702 0.0" rpy="0 0 0"/>
     <mass value="${vehicle_body_mass}"/>
     <inertia ixx="${vehicle_inertia_coef*114.688091}" iyy="${vehicle_inertia_coef*336.418835}" izz="${vehicle_inertia_coef*418.647558}" ixy="${vehicle_inertia_coef*0.010139}" iyz="${vehicle_inertia_coef*0.002956}" ixz="${-vehicle_inertia_coef*0.33997}"/>
@@ -199,5 +199,5 @@
     <origin xyz="0 0 0" rpy="1.57 0 0"/>
     <geometry>
-      <cylinder radius="0.16" length="0.05"/>
+      <cylinder radius="0.155" length="0.05"/>
     </geometry>
     <!-- ここから SDF の surface/friction -->
@@ -240,5 +240,5 @@
     <origin xyz="0 0 0" rpy="1.57 0 0"/>
     <geometry>
-      <cylinder radius="0.16" length="0.05"/>
+      <cylinder radius="0.155" length="0.05"/>
     </geometry>
     <!-- ここから SDF の surface/friction -->
@@ -281,5 +281,5 @@
     <origin xyz="0 0 0" rpy="1.57 0 0"/>
     <geometry>
-      <cylinder radius="0.16" length="0.05"/>
+      <cylinder radius="0.155" length="0.05"/>
     </geometry>
     <!-- ここから SDF の surface/friction -->
@@ -322,5 +322,5 @@
     <origin xyz="0 0 0" rpy="1.57 0 0"/>
     <geometry>
-      <cylinder radius="0.16" length="0.05"/>
+      <cylinder radius="0.155" length="0.05"/>
     </geometry>
     <!-- ここから SDF の surface/friction -->
@@ -344,5 +344,5 @@
 </link>
 <joint name="body" type="fixed">
-  <origin xyz="0 0 0.376" rpy="0 0 0"/>
+  <origin xyz="0 -0.05 0.376" rpy="0 0 0"/>
   <parent link="base_link"/>
   <child link="body_link"/>

Commit message: 202506261234

File: urdf/vehicle_4ws_real.xacro (robot description, xacro)
@@ -364,5 +364,5 @@
   <dynamics damping="${front_steering_damping}" friction="${front_steering_friction}"/>
   <axis xyz="0.0 0.0 1.0"/>
-  <limit upper="1.047" lower="-1.047" effort="100" velocity="100"/>
+  <limit upper="1.57" lower="-1.57" effort="200" velocity="200"/>
 </joint>
 <joint name="front_right_wheel" type="continuous">
@@ -388,5 +388,5 @@
   <dynamics damping="${front_steering_damping}" friction="${front_steering_friction}"/>
   <axis xyz="0.0 0.0 1.0"/>
-  <limit upper="1.047" lower="-1.047" effort="100" velocity="100"/>
+  <limit upper="1.57" lower="-1.57" effort="200" velocity="200"/>
 </joint>
 <joint name="front_left_wheel" type="continuous">

Commit message: 2025062712simulation

File: urdf/vehicle_4ws_real.xacro (robot description, xacro)
@@ -193,11 +193,7 @@
   </visual>
   <collision>
-    <!-- <origin xyz="-0.450031 0.34248 -0.150215" rpy="0 0 0"/> -->
-    <!-- <geometry>
-      <mesh filename="package://vehicle_4ws_description/meshes/new_wheel_1.stl" scale="0.001 0.001 0.001"/>
-    </geometry> -->
     <origin xyz="0 0 0" rpy="1.57 0 0"/>
     <geometry>
-      <cylinder radius="0.155" length="0.05"/>
+      <cylinder radius="0.153" length="0.05"/>
     </geometry>
     <!-- ここから SDF の surface/friction -->
@@ -240,5 +236,5 @@
     <origin xyz="0 0 0" rpy="1.57 0 0"/>
     <geometry>
-      <cylinder radius="0.155" length="0.05"/>
+      <cylinder radius="0.153" length="0.05"/>
     </geometry>
     <!-- ここから SDF の surface/friction -->
@@ -281,5 +277,5 @@
     <origin xyz="0 0 0" rpy="1.57 0 0"/>
     <geometry>
-      <cylinder radius="0.155" length="0.05"/>
+      <cylinder radius="0.153" length="0.05"/>
     </geometry>
     <!-- ここから SDF の surface/friction -->
@@ -322,5 +318,5 @@
     <origin xyz="0 0 0" rpy="1.57 0 0"/>
     <geometry>
-      <cylinder radius="0.155" length="0.05"/>
+      <cylinder radius="0.153" length="0.05"/>
     </geometry>
     <!-- ここから SDF の surface/friction -->

Commit message: デバッグ

File: urdf/vehicle_4ws_real.xacro (robot description, xacro)
@@ -402,13 +402,24 @@
   <axis xyz="0.0 1.0 -0.0"/>
 </joint>
-<joint name="rear_to_Rsteering" type="fixed">
+<!-- 後輪右ステア -->
+<joint name="rear_right_steering" type="revolute">
   <origin xyz="0.0 -0.4 -0.02" rpy="0 0 0"/>
   <parent link="v1_rear_1"/>
-  <child link="new_hinge_2"/>
-</joint>
-<joint name="rear_to_Lsteering" type="fixed">
+  <child  link="new_hinge_2"/>
+  <!-- ステア駆動時のダンピング・摩擦 -->
+  <dynamics damping="${steering_damping}" friction="${steering_friction}"/>
+  <!-- 回転軸は Z 方向 -->
+  <axis    xyz="0.0 0.0 1.0"/>
+  <!-- 可動範囲／トルク／速度制限 -->
+  <limit  lower="-1.57" upper="1.57" effort="200" velocity="200"/>
+</joint>
+<!-- 後輪左ステア -->
+<joint name="rear_left_steering" type="revolute">
   <origin xyz="0.0 0.4 -0.02" rpy="0 0 0"/>
   <parent link="v1_rear_1"/>
-  <child link="new_hinge_4"/>
+  <child  link="new_hinge_4"/>
+  <dynamics damping="${steering_damping}" friction="${steering_friction}"/>
+  <axis    xyz="0.0 0.0 1.0"/>
+  <limit  lower="-1.57" upper="1.57" effort="200" velocity="200"/>
 </joint>
 </robot>

Commit message: 202507030941

File: urdf/vehicle_4ws_real.xacro (robot description, xacro)
@@ -34,7 +34,7 @@
 <xacro:property name="rotational_joint_mu" value="0.001" />
 <xacro:property name="rotational_joint_friction" value="${rotational_joint_mu * gravitational_acceleration}" />
-<xacro:include filename="$(find vehicle_4ws_description)/urdf/materials.xacro" />
-<xacro:include filename="$(find vehicle_4ws_description)/urdf/vehicle_4ws.trans" />
-<xacro:include filename="$(find vehicle_4ws_description)/urdf/vehicle_4ws.gazebo" />
+<xacro:include filename="$(find 4ws_backstepping)/urdf/materials.xacro" />
+<xacro:include filename="$(find 4ws_backstepping)/urdf/vehicle_4ws.trans" />
+<xacro:include filename="$(find 4ws_backstepping)/urdf/vehicle_4ws.gazebo" />
 <link name="base_link"/>
 <link name="body_link">
@@ -47,5 +47,5 @@
     <origin xyz="0 0 -0.376" rpy="0 0 0"/>
     <geometry>
-      <mesh filename="package://vehicle_4ws_description/meshes/base_link.stl" scale="0.001 0.001 0.001"/>
+      <mesh filename="package://4ws_backstepping/meshes/base_link.stl" scale="0.001 0.001 0.001"/>
     </geometry>
     <material name="_"/>
@@ -54,5 +54,5 @@
     <origin xyz="0 0 -0.376" rpy="0 0 0"/>
     <geometry>
-      <mesh filename="package://vehicle_4ws_description/meshes/base_link.stl" scale="0.001 0.001 0.001"/>
+      <mesh filename="package://4ws_backstepping/meshes/base_link.stl" scale="0.001 0.001 0.001"/>
     </geometry>
   </collision>
@@ -67,5 +67,5 @@
     <origin xyz="0.44955 -0.05752 -0.376" rpy="0 0 0"/>
     <geometry>
-      <mesh filename="package://vehicle_4ws_description/meshes/v1_rear_1.stl" scale="0.001 0.001 0.001"/>
+      <mesh filename="package://4ws_backstepping/meshes/v1_rear_1.stl" scale="0.001 0.001 0.001"/>
     </geometry>
     <material name="_"/>
@@ -74,5 +74,5 @@
     <origin xyz="0.44955 -0.05752 -0.376" rpy="0 0 0"/>
     <geometry>
-      <mesh filename="package://vehicle_4ws_description/meshes/v1_rear_1.stl" scale="0.001 0.001 0.001"/>
+      <mesh filename="package://4ws_backstepping/meshes/v1_rear_1.stl" scale="0.001 0.001 0.001"/>
     </geometry>
   </collision>
@@ -87,5 +87,5 @@
     <origin xyz="-0.45045 -0.05752 -0.376" rpy="0 0 0"/>
     <geometry>
-      <mesh filename="package://vehicle_4ws_description/meshes/v1_front_1.stl" scale="0.001 0.001 0.001"/>
+      <mesh filename="package://4ws_backstepping/meshes/v1_front_1.stl" scale="0.001 0.001 0.001"/>
     </geometry>
     <material name="_"/>
@@ -94,5 +94,5 @@
     <origin xyz="-0.45045 -0.05752 -0.376" rpy="0 0 0"/>
     <geometry>
-      <mesh filename="package://vehicle_4ws_description/meshes/v1_front_1.stl" scale="0.001 0.001 0.001"/>
+      <mesh filename="package://4ws_backstepping/meshes/v1_front_1.stl" scale="0.001 0.001 0.001"/>
     </geometry>
   </collision>
@@ -107,5 +107,5 @@
     <origin xyz="-0.45045 0.34248 -0.356" rpy="0 0 0"/>
     <geometry>
-      <mesh filename="package://vehicle_4ws_description/meshes/new_hinge_1.stl" scale="0.001 0.001 0.001"/>
+      <mesh filename="package://4ws_backstepping/meshes/new_hinge_1.stl" scale="0.001 0.001 0.001"/>
     </geometry>
     <material name="_"/>
@@ -114,5 +114,5 @@
     <origin xyz="-0.45045 0.34248 -0.356" rpy="0 0 0"/>
     <geometry>
-      <mesh filename="package://vehicle_4ws_description/meshes/new_hinge_1.stl" scale="0.001 0.001 0.001"/>
+      <mesh filename="package://4ws_backstepping/meshes/new_hinge_1.stl" scale="0.001 0.001 0.001"/>
     </geometry>
   </collision>
@@ -127,5 +127,5 @@
     <origin xyz="-0.45045 -0.45752 -0.356" rpy="0 0 0"/>
     <geometry>
-      <mesh filename="package://vehicle_4ws_description/meshes/new_hinge_3.stl" scale="0.001 0.001 0.001"/>
+      <mesh filename="package://4ws_backstepping/meshes/new_hinge_3.stl" scale="0.001 0.001 0.001"/>
     </geometry>
     <material name="_"/>
@@ -134,5 +134,5 @@
     <origin xyz="-0.45045 -0.45752 -0.356" rpy="0 0 0"/>
     <geometry>
-      <mesh filename="package://vehicle_4ws_description/meshes/new_hinge_3.stl" scale="0.001 0.001 0.001"/>
+      <mesh filename="package://4ws_backstepping/meshes/new_hinge_3.stl" scale="0.001 0.001 0.001"/>
     </geometry>
   </collision>
@@ -147,5 +147,5 @@
     <origin xyz="0.44955 0.34248 -0.356" rpy="0 0 0"/>
     <geometry>
-      <mesh filename="package://vehicle_4ws_description/meshes/new_hinge_2.stl" scale="0.001 0.001 0.001"/>
+      <mesh filename="package://4ws_backstepping/meshes/new_hinge_2.stl" scale="0.001 0.001 0.001"/>
     </geometry>
     <material name="_"/>
@@ -154,5 +154,5 @@
     <origin xyz="0.44955 0.34248 -0.356" rpy="0 0 0"/>
     <geometry>
-      <mesh filename="package://vehicle_4ws_description/meshes/new_hinge_2.stl" scale="0.001 0.001 0.001"/>
+      <mesh filename="package://4ws_backstepping/meshes/new_hinge_2.stl" scale="0.001 0.001 0.001"/>
     </geometry>
   </collision>
@@ -167,5 +167,5 @@
     <origin xyz="0.44955 -0.45752 -0.356" rpy="0 0 0"/>
     <geometry>
-      <mesh filename="package://vehicle_4ws_description/meshes/new_hinge_4.stl" scale="0.001 0.001 0.001"/>
+      <mesh filename="package://4ws_backstepping/meshes/new_hinge_4.stl" scale="0.001 0.001 0.001"/>
     </geometry>
     <material name="_"/>
@@ -174,5 +174,5 @@
     <origin xyz="0.44955 -0.45752 -0.356" rpy="0 0 0"/>
     <geometry>
-      <mesh filename="package://vehicle_4ws_description/meshes/new_hinge_4.stl" scale="0.001 0.001 0.001"/>
+      <mesh filename="package://4ws_backstepping/meshes/new_hinge_4.stl" scale="0.001 0.001 0.001"/>
     </geometry>
   </collision>
@@ -188,5 +188,5 @@
     <origin xyz="-0.450031 0.34248 -0.150215" rpy="0 0 0"/>
     <geometry>
-      <mesh filename="package://vehicle_4ws_description/meshes/new_wheel_1.stl" scale="0.001 0.001 0.001"/>
+      <mesh filename="package://4ws_backstepping/meshes/new_wheel_1.stl" scale="0.001 0.001 0.001"/>
     </geometry>
     <material name="_"/>
@@ -225,5 +225,5 @@
     <origin xyz="0.449969 0.34248 -0.150215" rpy="0 0 0"/>
     <geometry>
-      <mesh filename="package://vehicle_4ws_description/meshes/new_wheel_2.stl" scale="0.001 0.001 0.001"/>
+      <mesh filename="package://4ws_backstepping/meshes/new_wheel_2.stl" scale="0.001 0.001 0.001"/>
     </geometry>
     <material name="_"/>
@@ -232,5 +232,5 @@
     <!-- <origin xyz="0.449969 0.34248 -0.150215" rpy="0 0 0"/>
     <geometry>
-      <mesh filename="package://vehicle_4ws_description/meshes/new_wheel_2.stl" scale="0.001 0.001 0.001"/>
+      <mesh filename="package://4ws_backstepping/meshes/new_wheel_2.stl" scale="0.001 0.001 0.001"/>
     </geometry> -->
     <origin xyz="0 0 0" rpy="1.57 0 0"/>
@@ -266,5 +266,5 @@
     <origin xyz="-0.450031 -0.45752 -0.150215" rpy="0 0 0"/>
     <geometry>
-      <mesh filename="package://vehicle_4ws_description/meshes/new_wheel_3.stl" scale="0.001 0.001 0.001"/>
+      <mesh filename="package://4ws_backstepping/meshes/new_wheel_3.stl" scale="0.001 0.001 0.001"/>
     </geometry>
     <material name="_"/>
@@ -273,5 +273,5 @@
     <!-- <origin xyz="-0.450031 -0.45752 -0.150215" rpy="0 0 0"/>
     <geometry>
-      <mesh filename="package://vehicle_4ws_description/meshes/new_wheel_3.stl" scale="0.001 0.001 0.001"/>
+      <mesh filename="package://4ws_backstepping/meshes/new_wheel_3.stl" scale="0.001 0.001 0.001"/>
     </geometry> -->
     <origin xyz="0 0 0" rpy="1.57 0 0"/>
@@ -307,5 +307,5 @@
     <origin xyz="0.449969 -0.45752 -0.150215" rpy="0 0 0"/>
     <geometry>
-      <mesh filename="package://vehicle_4ws_description/meshes/new_wheel_4.stl" scale="0.001 0.001 0.001"/>
+      <mesh filename="package://4ws_backstepping/meshes/new_wheel_4.stl" scale="0.001 0.001 0.001"/>
     </geometry>
     <material name="_"/>
@@ -314,5 +314,5 @@
     <!-- <origin xyz="0.449969 -0.45752 -0.150215" rpy="0 0 0"/>
     <geometry>
-      <mesh filename="package://vehicle_4ws_description/meshes/new_wheel_4.stl" scale="0.001 0.001 0.001"/>
+      <mesh filename="package://4ws_backstepping/meshes/new_wheel_4.stl" scale="0.001 0.001 0.001"/>
     </geometry> -->
     <origin xyz="0 0 0" rpy="1.57 0 0"/>

Commit message: パラメーター調整

File: urdf/vehicle_4ws_real.xacro (robot description, xacro)
@@ -10,6 +10,6 @@
 <xacro:property name="wheel_mass" value="4.639715839283939" />
 <!-- frontは受動車輪なので低めに設定 -->
-<xacro:property name="front_wheel_joint_damping" value="0.1"/>
-<xacro:property name="front_wheel_joint_mu" value="0.001" />
+<xacro:property name="front_wheel_joint_damping" value="0.0"/>
+<xacro:property name="front_wheel_joint_mu" value="0.000" />
 <xacro:property name="front_wheel_joint_friction" value="${front_wheel_joint_mu* gravitational_acceleration * wheel_mass  }" />
 <xacro:property name="front_steering_damping" value="5.0" />
@@ -17,17 +17,17 @@
 <xacro:property name="front_steering_friction" value="${front_steering_mu * gravitational_acceleration * 0.25*vehicle_body_mass}" />
 <!-- rearは駆動輪なので、入力以外で動かないように設定 -->
-<xacro:property name="wheel_joint_damping" value="0.2"/>
-<xacro:property name="wheel_joint_mu" value="0.05" />
-<xacro:property name="wheel_joint_friction" value="${wheel_joint_mu* gravitational_acceleration * wheel_mass }" />
-<xacro:property name="steering_damping" value="20.0" />
-<xacro:property name="steering_mu" value="0.01" />
-<xacro:property name="steering_friction" value="${steering_mu * gravitational_acceleration * 0.25*vehicle_body_mass}" />
+<xacro:property name="rear_wheel_joint_damping" value="0.0"/>
+<xacro:property name="rear_wheel_joint_mu" value="0.000" />
+<xacro:property name="rear_wheel_joint_friction" value="${rear_wheel_joint_mu* gravitational_acceleration * wheel_mass }" />
+<xacro:property name="rear_steering_damping" value="5.0" />
+<xacro:property name="rear_steering_mu" value="0.001" />
+<xacro:property name="rear_steering_friction" value="${rear_steering_mu * gravitational_acceleration * 0.25*vehicle_body_mass}" />
 <!-- wheelの接地面の摩擦などを定義 -->
 <xacro:property name="wheel_surface_mu1" value="5.0"/>
 <xacro:property name="wheel_surface_mu2" value="5.0" />
-<xacro:property name="wheel_kp" value="1e5" />
+<xacro:property name="wheel_kp" value="5e4" />
 <xacro:property name="wheel_kd" value="1.0" />
 <xacro:property name="wheel_minDepth" value="0.01" />
-<xacro:property name="wheel_maxVel" value="0.1" />
+<xacro:property name="wheel_maxVel" value="1.0" />
 <!-- rotationは共通 -->
 <xacro:property name="rotational_joint_damping" value="0.01" />
@@ -40,5 +40,5 @@
 <link name="body_link">
   <inertial>
-    <origin xyz="0.001411408730126027 0.05751189617802702 0.0" rpy="0 0 0"/>
+    <origin xyz="0.001411408730126027 0.05751189617802702 -0.05" rpy="0 0 0"/>
     <mass value="${vehicle_body_mass}"/>
     <inertia ixx="${vehicle_inertia_coef*114.688091}" iyy="${vehicle_inertia_coef*336.418835}" izz="${vehicle_inertia_coef*418.647558}" ixy="${vehicle_inertia_coef*0.010139}" iyz="${vehicle_inertia_coef*0.002956}" ixz="${-vehicle_inertia_coef*0.33997}"/>
@@ -374,5 +374,5 @@
   <parent link="new_hinge_2"/>
   <child link="new_wheel_2"/>
-  <dynamics damping="${wheel_joint_damping}" friction="${wheel_joint_friction}"/>
+  <dynamics damping="${rear_wheel_joint_damping}" friction="${rear_wheel_joint_friction}"/>
   <limit effort="500" velocity="500"/>
   <axis xyz="0.0 1.0 -0.0"/>
@@ -398,5 +398,5 @@
   <parent link="new_hinge_4"/>
   <child link="new_wheel_4"/>
-  <dynamics damping="${wheel_joint_damping}" friction="${wheel_joint_friction}"/>
+  <dynamics damping="${rear_wheel_joint_damping}" friction="${rear_wheel_joint_friction}"/>
   <limit effort="500" velocity="500"/>
   <axis xyz="0.0 1.0 -0.0"/>
@@ -408,5 +408,5 @@
   <child  link="new_hinge_2"/>
   <!-- ステア駆動時のダンピング・摩擦 -->
-  <dynamics damping="${steering_damping}" friction="${steering_friction}"/>
+  <dynamics damping="${rear_steering_damping}" friction="${rear_steering_friction}"/>
   <!-- 回転軸は Z 方向 -->
   <axis    xyz="0.0 0.0 1.0"/>
@@ -419,5 +419,5 @@
   <parent link="v1_rear_1"/>
   <child  link="new_hinge_4"/>
-  <dynamics damping="${steering_damping}" friction="${steering_friction}"/>
+  <dynamics damping="${rear_steering_damping}" friction="${rear_steering_friction}"/>
   <axis    xyz="0.0 0.0 1.0"/>
   <limit  lower="-1.57" upper="1.57" effort="200" velocity="200"/>

Commit message: 完走_d0.029

File: urdf/vehicle_4ws_real.xacro (robot description, xacro)
@@ -10,20 +10,20 @@
 <xacro:property name="wheel_mass" value="4.639715839283939" />
 <!-- frontは受動車輪なので低めに設定 -->
-<xacro:property name="front_wheel_joint_damping" value="0.0"/>
-<xacro:property name="front_wheel_joint_mu" value="0.000" />
+<xacro:property name="front_wheel_joint_damping" value="1.0"/>
+<xacro:property name="front_wheel_joint_mu" value="0.1" />
 <xacro:property name="front_wheel_joint_friction" value="${front_wheel_joint_mu* gravitational_acceleration * wheel_mass  }" />
-<xacro:property name="front_steering_damping" value="5.0" />
+<xacro:property name="front_steering_damping" value="3.0" />
 <xacro:property name="front_steering_mu" value="0.001" />
 <xacro:property name="front_steering_friction" value="${front_steering_mu * gravitational_acceleration * 0.25*vehicle_body_mass}" />
 <!-- rearは駆動輪なので、入力以外で動かないように設定 -->
-<xacro:property name="rear_wheel_joint_damping" value="0.0"/>
-<xacro:property name="rear_wheel_joint_mu" value="0.000" />
+<xacro:property name="rear_wheel_joint_damping" value="1.0"/>
+<xacro:property name="rear_wheel_joint_mu" value="0.1" />
 <xacro:property name="rear_wheel_joint_friction" value="${rear_wheel_joint_mu* gravitational_acceleration * wheel_mass }" />
-<xacro:property name="rear_steering_damping" value="5.0" />
+<xacro:property name="rear_steering_damping" value="3.0" />
 <xacro:property name="rear_steering_mu" value="0.001" />
 <xacro:property name="rear_steering_friction" value="${rear_steering_mu * gravitational_acceleration * 0.25*vehicle_body_mass}" />
 <!-- wheelの接地面の摩擦などを定義 -->
-<xacro:property name="wheel_surface_mu1" value="5.0"/>
-<xacro:property name="wheel_surface_mu2" value="5.0" />
+<xacro:property name="wheel_surface_mu1" value="4.0"/>
+<xacro:property name="wheel_surface_mu2" value="4.0" />
 <xacro:property name="wheel_kp" value="5e4" />
 <xacro:property name="wheel_kd" value="1.0" />

Commit message: 制御点3つ

File: urdf/vehicle_4ws_real.xacro (robot description, xacro)
@@ -24,6 +24,6 @@
 <xacro:property name="rear_steering_friction" value="${rear_steering_mu * gravitational_acceleration * 0.25*vehicle_body_mass}" />
 <!-- wheelの接地面の摩擦などを定義 -->
-<xacro:property name="wheel_surface_mu1" value="4.0"/>
-<xacro:property name="wheel_surface_mu2" value="4.0" />
+<xacro:property name="wheel_surface_mu1" value="2.0"/>
+<xacro:property name="wheel_surface_mu2" value="2.0" />
 <xacro:property name="wheel_kp" value="5e4" />
 <xacro:property name="wheel_kd" value="1.0" />

Commit message: 完走_d0.009

File: urdf/vehicle_4ws_real.xacro (robot description, xacro)
@@ -24,6 +24,6 @@
 <xacro:property name="rear_steering_friction" value="${rear_steering_mu * gravitational_acceleration * 0.25*vehicle_body_mass}" />
 <!-- wheelの接地面の摩擦などを定義 -->
-<xacro:property name="wheel_surface_mu1" value="2.0"/>
-<xacro:property name="wheel_surface_mu2" value="2.0" />
+<xacro:property name="wheel_surface_mu1" value="3.0"/>
+<xacro:property name="wheel_surface_mu2" value="3.0" />
 <xacro:property name="wheel_kp" value="5e4" />
 <xacro:property name="wheel_kd" value="1.0" />

Commit message: d_0.0023,mb=100

File: urdf/vehicle_4ws_real.xacro (robot description, xacro)
@@ -2,9 +2,9 @@
 <robot name="vehicle_4ws" xmlns:xacro="http://www.ros.org/wiki/xacro">
 <xacro:property name="PI" value="3.1415926535897932384626433832795028841971" />
-<xacro:property name="gravitational_acceleration" value="9.8" />
+<xacro:property name="gravitational_acceleration" value="9.80665" />
 <xacro:property name="vehicle1_Yaw" value="-PI/4" />
 <!-- 荷台と連結点のmass -->
 <xacro:property name="fusion_vehicle_body_mass" value="2113.272311120373" />
-<xacro:property name="vehicle_body_mass" value="313.272311120373" />
+<xacro:property name="vehicle_body_mass" value="100" />
 <xacro:property name="vehicle_inertia_coef" value="${vehicle_body_mass/fusion_vehicle_body_mass}" />
 <xacro:property name="wheel_mass" value="4.639715839283939" />
@@ -24,6 +24,6 @@
 <xacro:property name="rear_steering_friction" value="${rear_steering_mu * gravitational_acceleration * 0.25*vehicle_body_mass}" />
 <!-- wheelの接地面の摩擦などを定義 -->
-<xacro:property name="wheel_surface_mu1" value="3.0"/>
-<xacro:property name="wheel_surface_mu2" value="3.0" />
+<xacro:property name="wheel_surface_mu1" value="1.0"/>
+<xacro:property name="wheel_surface_mu2" value="1.0" />
 <xacro:property name="wheel_kp" value="5e4" />
 <xacro:property name="wheel_kd" value="1.0" />
