Commit message: d_0.0023

File: urdf/vehicle_4ws_real.xacro (robot description, xacro)
@@ -40,10 +40,10 @@
 <link name="body_link">
   <inertial>
-    <origin xyz="0.001411408730126027 0.05751189617802702 -0.05" rpy="0 0 0"/>
+    <origin xyz="0.001411408730126027 0.0 -0.05" rpy="0 0 0"/>
     <mass value="${vehicle_body_mass}"/>
     <inertia ixx="${vehicle_inertia_coef*114.688091}" iyy="${vehicle_inertia_coef*336.418835}" izz="${vehicle_inertia_coef*418.647558}" ixy="${vehicle_inertia_coef*0.010139}" iyz="${vehicle_inertia_coef*0.002956}" ixz="${-vehicle_inertia_coef*0.33997}"/>
   </inertial>
   <visual>
-    <origin xyz="0 0 -0.376" rpy="0 0 0"/>
+    <origin xyz="0 -0.05 -0.376" rpy="0 0 0"/>
     <geometry>
       <mesh filename="package://4ws_backstepping/meshes/base_link.stl" scale="0.001 0.001 0.001"/>
@@ -52,5 +52,5 @@
   </visual>
   <collision>
-    <origin xyz="0 0 -0.376" rpy="0 0 0"/>
+    <origin xyz="0 -0.05 -0.376" rpy="0 0 0"/>
     <geometry>
       <mesh filename="package://4ws_backstepping/meshes/base_link.stl" scale="0.001 0.001 0.001"/>
@@ -65,5 +65,5 @@
   </inertial>
   <visual>
-    <origin xyz="0.44955 -0.05752 -0.376" rpy="0 0 0"/>
+    <origin xyz="0.44955 -0.10752 -0.376" rpy="0 0 0"/>
     <geometry>
       <mesh filename="package://4ws_backstepping/meshes/v1_rear_1.stl" scale="0.001 0.001 0.001"/>
@@ -72,5 +72,5 @@
   </visual>
   <collision>
-    <origin xyz="0.44955 -0.05752 -0.376" rpy="0 0 0"/>
+    <origin xyz="0.44955 -0.10752 -0.376" rpy="0 0 0"/>
     <geometry>
       <mesh filename="package://4ws_backstepping/meshes/v1_rear_1.stl" scale="0.001 0.001 0.001"/>
@@ -85,5 +85,5 @@
   </inertial>
   <visual>
-    <origin xyz="-0.45045 -0.05752 -0.376" rpy="0 0 0"/>
+    <origin xyz="-0.45045 -0.10752 -0.376" rpy="0 0 0"/>
     <geometry>
       <mesh filename="package://4ws_backstepping/meshes/v1_front_1.stl" scale="0.001 0.001 0.001"/>
@@ -92,5 +92,5 @@
   </visual>
   <collision>
-    <origin xyz="-0.45045 -0.05752 -0.376" rpy="0 0 0"/>
+    <origin xyz="-0.45045 -0.10752 -0.376" rpy="0 0 0"/>
     <geometry>
       <mesh filename="package://4ws_backstepping/meshes/v1_front_1.stl" scale="0.001 0.001 0.001"/>
@@ -105,5 +105,5 @@
   </inertial>
   <visual>
-    <origin xyz="-0.45045 0.34248 -0.356" rpy="0 0 0"/>
+    <origin xyz="-0.45045 0.29248 -0.356" rpy="0 0 0"/>
     <geometry>
       <mesh filename="package://4ws_backstepping/meshes/new_hinge_1.stl" scale="0.001 0.001 0.001"/>
@@ -112,5 +112,5 @@
   </visual>
   <collision>
-    <origin xyz="-0.45045 0.34248 -0.356" rpy="0 0 0"/>
+    <origin xyz="-0.45045 0.29248 -0.356" rpy="0 0 0"/>
     <geometry>
       <mesh filename="package://4ws_backstepping/meshes/new_hinge_1.stl" scale="0.001 0.001 0.001"/>
@@ -125,5 +125,5 @@
   </inertial>
   <visual>
-    <origin xyz="-0.45045 -0.45752 -0.356" rpy="0 0 0"/>
+    <origin xyz="-0.45045 -0.50752 -0.356" rpy="0 0 0"/>
     <geometry>
       <mesh filename="package://4ws_backstepping/meshes/new_hinge_3.stl" scale="0.001 0.001 0.001"/>
@@ -132,5 +132,5 @@
   </visual>
   <collision>
-    <origin xyz="-0.45045 -0.45752 -0.356" rpy="0 0 0"/>
+    <origin xyz="-0.45045 -0.50752 -0.356" rpy="0 0 0"/>
     <geometry>
       <mesh filename="package://4ws_backstepping/meshes/new_hinge_3.stl" scale="0.001 0.001 0.001"/>
@@ -145,5 +145,5 @@
   </inertial>
   <visual>
-    <origin xyz="0.44955 0.34248 -0.356" rpy="0 0 0"/>
+    <origin xyz="0.44955 0.29248 -0.356" rpy="0 0 0"/>
     <geometry>
       <mesh filename="package://4ws_backstepping/meshes/new_hinge_2.stl" scale="0.001 0.001 0.001"/>
@@ -152,5 +152,5 @@
   </visual>
   <collision>
-    <origin xyz="0.44955 0.34248 -0.356" rpy="0 0 0"/>
+    <origin xyz="0.44955 0.29248 -0.356" rpy="0 0 0"/>
     <geometry>
       <mesh filename="package://4ws_backstepping/meshes/new_hinge_2.stl" scale="0.001 0.001 0.001"/>
@@ -165,5 +165,5 @@
   </inertial>
   <visual>
-    <origin xyz="0.44955 -0.45752 -0.356" rpy="0 0 0"/>
+    <origin xyz="0.44955 -0.50752 -0.356" rpy="0 0 0"/>
     <geometry>
       <mesh filename="package://4ws_backstepping/meshes/new_hinge_4.stl" scale="0.001 0.001 0.001"/>
@@ -172,5 +172,5 @@
   </visual>
   <collision>
-    <origin xyz="0.44955 -0.45752 -0.356" rpy="0 0 0"/>
+    <origin xyz="0.44955 -0.50752 -0.356" rpy="0 0 0"/>
     <geometry>
       <mesh filename="package://4ws_backstepping/meshes/new_hinge_4.stl" scale="0.001 0.001 0.001"/>
@@ -186,5 +186,5 @@
   </inertial>
   <visual>
-    <origin xyz="-0.450031 0.34248 -0.150215" rpy="0 0 0"/>
+    <origin xyz="-0.450031 0.29248 -0.150215" rpy="0 0 0"/>
     <geometry>
       <mesh filename="package://4ws_backstepping/meshes/new_wheel_1.stl" scale="0.001 0.001 0.001"/>
@@ -223,5 +223,5 @@
   </inertial>
   <visual>
-    <origin xyz="0.449969 0.34248 -0.150215" rpy="0 0 0"/>
+    <origin xyz="0.449969 0.29248 -0.150215" rpy="0 0 0"/>
     <geometry>
       <mesh filename="package://4ws_backstepping/meshes/new_wheel_2.stl" scale="0.001 0.001 0.001"/>
@@ -230,5 +230,5 @@
   </visual>
   <collision>
-    <!-- <origin xyz="0.449969 0.34248 -0.150215" rpy="0 0 0"/>
+    <!-- <origin xyz="0.449969 0.29248 -0.150215" rpy="0 0 0"/>
     <geometry>
       <mesh filename="package://4ws_backstepping/meshes/new_wheel_2.stl" scale="0.001 0.001 0.001"/>
@@ -264,5 +264,5 @@
   </inertial>
   <visual>
-    <origin xyz="-0.450031 -0.45752 -0.150215" rpy="0 0 0"/>
+    <origin xyz="-0.450031 -0.50752 -0.150215" rpy="0 0 0"/>
     <geometry>
       <mesh filename="package://4ws_backstepping/meshes/new_wheel_3.stl" scale="0.001 0.001 0.001"/>
@@ -271,5 +271,5 @@
   </visual>
   <collision>
-    <!-- <origin xyz="-0.450031 -0.45752 -0.150215" rpy="0 0 0"/>
+    <!-- <origin xyz="-0.450031 -0.50752 -0.150215" rpy="0 0 0"/>
     <geometry>
       <mesh filename="package://4ws_backstepping/meshes/new_wheel_3.stl" scale="0.001 0.001 0.001"/>
@@ -305,5 +305,5 @@
   </inertial>
   <visual>
-    <origin xyz="0.449969 -0.45752 -0.150215" rpy="0 0 0"/>
+    <origin xyz="0.449969 -0.50752 -0.150215" rpy="0 0 0"/>
     <geometry>
       <mesh filename="package://4ws_backstepping/meshes/new_wheel_4.stl" scale="0.001 0.001 0.001"/>
@@ -312,5 +312,5 @@
   </visual>
   <collision>
-    <!-- <origin xyz="0.449969 -0.45752 -0.150215" rpy="0 0 0"/>
+    <!-- <origin xyz="0.449969 -0.50752 -0.150215" rpy="0 0 0"/>
     <geometry>
       <mesh filename="package://4ws_backstepping/meshes/new_wheel_4.stl" scale="0.001 0.001 0.001"/>

Commit message: d_0.0019_20250724

File: urdf/vehicle_4ws_real.xacro (robot description, xacro)
@@ -8,4 +8,7 @@
 <xacro:property name="vehicle_body_mass" value="100" />
 <xacro:property name="vehicle_inertia_coef" value="${vehicle_body_mass/fusion_vehicle_body_mass}" />
+<xacro:property name="fusion_wheel_mass" value="4.639715839283939" />
+<xacro:property name="vehicle_wheel_mass" value="12" />
+<xacro:property name="wheel_inertia_coef" value="${vehicle_body_mass/fusion_vehicle_body_mass}" />
 <xacro:property name="wheel_mass" value="4.639715839283939" />
 <!-- frontは受動車輪なので低めに設定 -->

Commit message: 20250724

File: urdf/vehicle_4ws_real.xacro (robot description, xacro)
@@ -16,5 +16,5 @@
 <xacro:property name="front_wheel_joint_mu" value="0.1" />
 <xacro:property name="front_wheel_joint_friction" value="${front_wheel_joint_mu* gravitational_acceleration * wheel_mass  }" />
-<xacro:property name="front_steering_damping" value="3.0" />
+<xacro:property name="front_steering_damping" value="1.0" />
 <xacro:property name="front_steering_mu" value="0.001" />
 <xacro:property name="front_steering_friction" value="${front_steering_mu * gravitational_acceleration * 0.25*vehicle_body_mass}" />
@@ -23,5 +23,5 @@
 <xacro:property name="rear_wheel_joint_mu" value="0.1" />
 <xacro:property name="rear_wheel_joint_friction" value="${rear_wheel_joint_mu* gravitational_acceleration * wheel_mass }" />
-<xacro:property name="rear_steering_damping" value="3.0" />
+<xacro:property name="rear_steering_damping" value="1.0" />
 <xacro:property name="rear_steering_mu" value="0.001" />
 <xacro:property name="rear_steering_friction" value="${rear_steering_mu * gravitational_acceleration * 0.25*vehicle_body_mass}" />

Commit message: タイヤ重量変更

File: urdf/vehicle_4ws_real.xacro (robot description, xacro)
@@ -8,8 +8,14 @@
 <xacro:property name="vehicle_body_mass" value="100" />
 <xacro:property name="vehicle_inertia_coef" value="${vehicle_body_mass/fusion_vehicle_body_mass}" />
+<!-- 車輪のmass -->
 <xacro:property name="fusion_wheel_mass" value="4.639715839283939" />
 <xacro:property name="vehicle_wheel_mass" value="12" />
-<xacro:property name="wheel_inertia_coef" value="${vehicle_body_mass/fusion_vehicle_body_mass}" />
+<xacro:property name="wheel_inertia_coef" value="${vehicle_wheel_mass/fusion_wheel_mass}" />
 <xacro:property name="wheel_mass" value="4.639715839283939" />
+<!-- ステアリングのmass -->
+<xacro:property name="fusion_hinge_mass" value="4.639715839283939" />
+<xacro:property name="vehicle_hinge_mass" value="12" />
+<xacro:property name="hinge_inertia_coef" value="${vehicle_hinge_mass/fusion_hinge_mass}" />
+<xacro:property name="hinge_mass" value="4.639715839283939" />
 <!-- frontは受動車輪なので低めに設定 -->
 <xacro:property name="front_wheel_joint_damping" value="1.0"/>
@@ -185,6 +191,6 @@
   <inertial>
     <origin xyz="3.1709373395083507e-05 2.540692010666312e-07 0.00021681028363659816" rpy="0 0 0"/>
-    <mass value="4.639715839283939"/>
-    <inertia ixx="0.029034" iyy="0.053334" izz="0.029034" ixy="-0.0" iyz="0.0" ixz="0.0"/>
+    <mass value="${vehicle_wheel_mass}"/>
+    <inertia ixx="${wheel_inertia_coef*0.029034}" iyy="${wheel_inertia_coef*0.053334}" izz="${wheel_inertia_coef*0.029034}" ixy="-0.0" iyz="0.0" ixz="0.0"/>
   </inertial>
   <visual>
@@ -222,6 +228,6 @@
   <inertial>
     <origin xyz="3.1709373397914575e-05 2.5406927345317243e-07 0.00021681028363673693" rpy="0 0 0"/>
-    <mass value="4.639715839283939"/>
-    <inertia ixx="0.029034" iyy="0.053334" izz="0.029034" ixy="0.0" iyz="0.0" ixz="0.0"/>
+    <mass value="${vehicle_wheel_mass}"/>
+    <inertia ixx="${wheel_inertia_coef*0.029034}" iyy="${wheel_inertia_coef*0.053334}" izz="${wheel_inertia_coef*0.029034}"  ixy="0.0" iyz="0.0" ixz="0.0"/>
   </inertial>
   <visual>
@@ -263,6 +269,6 @@
   <inertial>
     <origin xyz="3.1709373395083507e-05 2.540692015662316e-07 0.00021681028363579324" rpy="0 0 0"/>
-    <mass value="4.639715839283939"/>
-    <inertia ixx="0.029034" iyy="0.053334" izz="0.029034" ixy="0.0" iyz="0.0" ixz="0.0"/>
+    <mass value="${vehicle_wheel_mass}"/>
+    <inertia ixx="${wheel_inertia_coef*0.029034}" iyy="${wheel_inertia_coef*0.053334}" izz="${wheel_inertia_coef*0.029034}"  ixy="0.0" iyz="0.0" ixz="0.0"/>
   </inertial>
   <visual>
@@ -304,6 +310,6 @@
   <inertial>
     <origin xyz="3.170937339708191e-05 2.540692737307282e-07 0.00021681028363593202" rpy="0 0 0"/>
-    <mass value="4.639715839283939"/>
-    <inertia ixx="0.029034" iyy="0.053334" izz="0.029034" ixy="0.0" iyz="0.0" ixz="0.0"/>
+    <mass value="${vehicle_wheel_mass}"/>
+    <inertia ixx="${wheel_inertia_coef*0.029034}" iyy="${wheel_inertia_coef*0.053334}" izz="${wheel_inertia_coef*0.029034}"  ixy="0.0" iyz="0.0" ixz="0.0"/>
   </inertial>
   <visual>

Commit message: d0.00105_20250726

File: urdf/vehicle_4ws_real.xacro (robot description, xacro)
@@ -114,5 +114,5 @@
   </inertial>
   <visual>
-    <origin xyz="-0.45045 0.29248 -0.356" rpy="0 0 0"/>
+    <origin xyz="-0.45045 0.34248 -0.356" rpy="0 0 0"/>
     <geometry>
       <mesh filename="package://4ws_backstepping/meshes/new_hinge_1.stl" scale="0.001 0.001 0.001"/>
@@ -134,5 +134,5 @@
   </inertial>
   <visual>
-    <origin xyz="-0.45045 -0.50752 -0.356" rpy="0 0 0"/>
+    <origin xyz="-0.45045 -0.45752 -0.356" rpy="0 0 0"/>
     <geometry>
       <mesh filename="package://4ws_backstepping/meshes/new_hinge_3.stl" scale="0.001 0.001 0.001"/>
@@ -154,5 +154,5 @@
   </inertial>
   <visual>
-    <origin xyz="0.44955 0.29248 -0.356" rpy="0 0 0"/>
+    <origin xyz="0.44955 0.34248 -0.356" rpy="0 0 0"/>
     <geometry>
       <mesh filename="package://4ws_backstepping/meshes/new_hinge_2.stl" scale="0.001 0.001 0.001"/>
@@ -174,5 +174,5 @@
   </inertial>
   <visual>
-    <origin xyz="0.44955 -0.50752 -0.356" rpy="0 0 0"/>
+    <origin xyz="0.44955 -0.45752 -0.356" rpy="0 0 0"/>
     <geometry>
       <mesh filename="package://4ws_backstepping/meshes/new_hinge_4.stl" scale="0.001 0.001 0.001"/>
@@ -195,5 +195,5 @@
   </inertial>
   <visual>
-    <origin xyz="-0.450031 0.29248 -0.150215" rpy="0 0 0"/>
+    <origin xyz="-0.450031 0.34248 -0.150215" rpy="0 0 0"/>
     <geometry>
       <mesh filename="package://4ws_backstepping/meshes/new_wheel_1.stl" scale="0.001 0.001 0.001"/>
@@ -232,5 +232,5 @@
   </inertial>
   <visual>
-    <origin xyz="0.449969 0.29248 -0.150215" rpy="0 0 0"/>
+    <origin xyz="0.449969 0.34248 -0.150215" rpy="0 0 0"/>
     <geometry>
       <mesh filename="package://4ws_backstepping/meshes/new_wheel_2.stl" scale="0.001 0.001 0.001"/>
@@ -273,5 +273,5 @@
   </inertial>
   <visual>
-    <origin xyz="-0.450031 -0.50752 -0.150215" rpy="0 0 0"/>
+    <origin xyz="-0.450031 -0.45752 -0.150215" rpy="0 0 0"/>
     <geometry>
       <mesh filename="package://4ws_backstepping/meshes/new_wheel_3.stl" scale="0.001 0.001 0.001"/>
@@ -314,5 +314,5 @@
   </inertial>
   <visual>
-    <origin xyz="0.449969 -0.50752 -0.150215" rpy="0 0 0"/>
+    <origin xyz="0.449969 -0.45752 -0.150215" rpy="0 0 0"/>
     <geometry>
       <mesh filename="package://4ws_backstepping/meshes/new_wheel_4.stl" scale="0.001 0.001 0.001"/>
@@ -349,5 +349,5 @@
 </link>
 <joint name="body" type="fixed">
-  <origin xyz="0 -0.05 0.376" rpy="0 0 0"/>
+  <origin xyz="0 0 0.376" rpy="0 0 0"/>
   <parent link="base_link"/>
   <child link="body_link"/>
@@ -364,5 +364,5 @@
 </joint>
 <joint name="front_right_steering" type="revolute">
-  <origin xyz="0.0 -0.4 -0.02" rpy="0 0 0"/>
+  <origin xyz="0.0 -0.45 -0.02" rpy="0 0 0"/>
   <parent link="v1_front_1"/>
   <child link="new_hinge_1"/>
@@ -388,5 +388,5 @@
 </joint>
 <joint name="front_left_steering" type="revolute">
-  <origin xyz="0.0 0.4 -0.02" rpy="0 0 0"/>
+  <origin xyz="0.0 0.35 -0.02" rpy="0 0 0"/>
   <parent link="v1_front_1"/>
   <child link="new_hinge_3"/>
@@ -413,5 +413,5 @@
 <!-- 後輪右ステア -->
 <joint name="rear_right_steering" type="revolute">
-  <origin xyz="0.0 -0.4 -0.02" rpy="0 0 0"/>
+  <origin xyz="0.0 -0.45 -0.02" rpy="0 0 0"/>
   <parent link="v1_rear_1"/>
   <child  link="new_hinge_2"/>
@@ -425,5 +425,5 @@
 <!-- 後輪左ステア -->
 <joint name="rear_left_steering" type="revolute">
-  <origin xyz="0.0 0.4 -0.02" rpy="0 0 0"/>
+  <origin xyz="0.0 0.35 -0.02" rpy="0 0 0"/>
   <parent link="v1_rear_1"/>
   <child  link="new_hinge_4"/>

Commit message: wheelとhingeの質量を12kgに変更

File: urdf/vehicle_4ws_real.xacro (robot description, xacro)
@@ -110,6 +110,6 @@
   <inertial>
     <origin xyz="-6.714468377522209e-05 2.5406917214532143e-07 -0.11523004751915897" rpy="0 0 0"/>
-    <mass value="4.884144703315957"/>
-    <inertia ixx="0.039519" iyy="0.032652" izz="0.021551" ixy="0.0" iyz="0.0" ixz="-3e-05"/>
+    <mass value="${vehicle_hinge_mass}"/>
+    <inertia ixx="${hinge_inertia_coef*0.039519}" iyy="${hinge_inertia_coef*0.032652}" izz="${hinge_inertia_coef*0.021551}" ixy="0.0" iyz="0.0" ixz="-3e-05"/>
   </inertial>
   <visual>
@@ -130,6 +130,6 @@
   <inertial>
     <origin xyz="-6.714468377522209e-05 2.5406917258941064e-07 -0.11523004751915977" rpy="0 0 0"/>
-    <mass value="4.884144703315957"/>
-    <inertia ixx="0.039519" iyy="0.032652" izz="0.021551" ixy="-0.0" iyz="0.0" ixz="-3e-05"/>
+    <mass value="${vehicle_hinge_mass}"/>
+    <inertia ixx="${hinge_inertia_coef*0.039519}" iyy="${hinge_inertia_coef*0.032652}" izz="${hinge_inertia_coef*0.021551}" ixy="-0.0" iyz="0.0" ixz="-3e-05"/>
   </inertial>
   <visual>
@@ -150,6 +150,6 @@
   <inertial>
     <origin xyz="-6.714468377322369e-05 2.540692444763515e-07 -0.1152300475191588" rpy="0 0 0"/>
-    <mass value="4.884144703315957"/>
-    <inertia ixx="0.039519" iyy="0.032652" izz="0.021551" ixy="0.0" iyz="0.0" ixz="-3e-05"/>
+    <mass value="${vehicle_hinge_mass}"/>
+    <inertia ixx="${hinge_inertia_coef*0.039519}" iyy="${hinge_inertia_coef*0.032652}" izz="${hinge_inertia_coef*0.021551}" ixy="0.0" iyz="0.0" ixz="-3e-05"/>
   </inertial>
   <visual>
@@ -170,6 +170,6 @@
   <inertial>
     <origin xyz="-6.714468377405636e-05 2.5406924475390724e-07 -0.11523004751915963" rpy="0 0 0"/>
-    <mass value="4.884144703315957"/>
-    <inertia ixx="0.039519" iyy="0.032652" izz="0.021551" ixy="0.0" iyz="0.0" ixz="-3e-05"/>
+    <mass value="${vehicle_hinge_mass}"/>
+    <inertia ixx="${hinge_inertia_coef*0.039519}" iyy="${hinge_inertia_coef*0.032652}" izz="${hinge_inertia_coef*0.021551}" ixy="0.0" iyz="0.0" ixz="-3e-05"/>
   </inertial>
   <visual>

Commit message: タイヤ8KG

File: urdf/vehicle_4ws_real.xacro (robot description, xacro)
@@ -10,5 +10,5 @@
 <!-- 車輪のmass -->
 <xacro:property name="fusion_wheel_mass" value="4.639715839283939" />
-<xacro:property name="vehicle_wheel_mass" value="12" />
+<xacro:property name="vehicle_wheel_mass" value="8" />
 <xacro:property name="wheel_inertia_coef" value="${vehicle_wheel_mass/fusion_wheel_mass}" />
 <xacro:property name="wheel_mass" value="4.639715839283939" />

File: urdf/vehicle_4ws_real_hill.xacro (robot description, xacro)
@@ -15,5 +15,5 @@
 <!-- ステアリングのmass -->
 <xacro:property name="fusion_hinge_mass" value="4.639715839283939" />
-<xacro:property name="vehicle_hinge_mass" value="12" />
+<xacro:property name="vehicle_hinge_mass" value="8" />
 <xacro:property name="hinge_inertia_coef" value="${vehicle_hinge_mass/fusion_hinge_mass}" />
 <xacro:property name="hinge_mass" value="4.639715839283939" />
@@ -376,5 +376,5 @@
   <child link="new_wheel_1"/>
   <dynamics damping="${front_wheel_joint_damping}" friction="${front_wheel_joint_friction}"/>
-  <limit effort="500" velocity="500"/>
+  <limit effort="100" velocity="100"/>
   <axis xyz="0.0 1.0 -0.0"/>
 </joint>
@@ -384,5 +384,5 @@
   <child link="new_wheel_2"/>
   <dynamics damping="${rear_wheel_joint_damping}" friction="${rear_wheel_joint_friction}"/>
-  <limit effort="500" velocity="500"/>
+  <limit effort="100" velocity="100"/>
   <axis xyz="0.0 1.0 -0.0"/>
 </joint>
@@ -400,5 +400,5 @@
   <child link="new_wheel_3"/>
   <dynamics damping="${front_wheel_joint_damping}" friction="${front_wheel_joint_friction}"/>
-  <limit effort="500" velocity="500"/>
+  <limit effort="100" velocity="100"/>
   <axis xyz="0.0 1.0 -0.0"/>
 </joint>
@@ -408,5 +408,5 @@
   <child link="new_wheel_4"/>
   <dynamics damping="${rear_wheel_joint_damping}" friction="${rear_wheel_joint_friction}"/>
-  <limit effort="500" velocity="500"/>
+  <limit effort="100" velocity="100"/>
   <axis xyz="0.0 1.0 -0.0"/>
 </joint>
