Commit message: ゲイン変更

File: urdf/vehicle_4ws_real_hill.xacro (robot description, xacro)
@@ -24,6 +24,6 @@
 <xacro:property name="rear_steering_friction" value="${rear_steering_mu * gravitational_acceleration * 0.25*vehicle_body_mass}" />
 <!-- wheelの接地面の摩擦などを定義 -->
-<xacro:property name="wheel_surface_mu1" value="1.0"/>
-<xacro:property name="wheel_surface_mu2" value="1.0" />
+<xacro:property name="wheel_surface_mu1" value="2.0"/>
+<xacro:property name="wheel_surface_mu2" value="2.0" />
 <xacro:property name="wheel_kp" value="5e4" />
 <xacro:property name="wheel_kd" value="1.0" />
@@ -40,10 +40,10 @@
 <link name="body_link">
   <inertial>
-    <origin xyz="0.001411408730126027 0.05751189617802702 -0.05" rpy="0 0 0"/>
+    <origin xyz="0.001411408730126027 0.0 -0.05" rpy="0 0 0"/>
     <mass value="${vehicle_body_mass}"/>
     <inertia ixx="${vehicle_inertia_coef*114.688091}" iyy="${vehicle_inertia_coef*336.418835}" izz="${vehicle_inertia_coef*418.647558}" ixy="${vehicle_inertia_coef*0.010139}" iyz="${vehicle_inertia_coef*0.002956}" ixz="${-vehicle_inertia_coef*0.33997}"/>
   </inertial>
   <visual>
-    <origin xyz="0 0 -0.376" rpy="0 0 0"/>
+    <origin xyz="0 -0.05 -0.376" rpy="0 0 0"/>
     <geometry>
       <mesh filename="package://4ws_backstepping/meshes/base_link.stl" scale="0.001 0.001 0.001"/>
@@ -52,5 +52,5 @@
   </visual>
   <collision>
-    <origin xyz="0 0 -0.376" rpy="0 0 0"/>
+    <origin xyz="0 -0.05 -0.376" rpy="0 0 0"/>
     <geometry>
       <mesh filename="package://4ws_backstepping/meshes/base_link.stl" scale="0.001 0.001 0.001"/>
@@ -60,10 +60,10 @@
 <link name="v1_rear_1">
   <inertial>
-    <origin xyz="2.514264385022891e-07 2.540692383215526e-07 -0.014912246259012996" rpy="0 0 0"/>
+    <origin xyz="2.514264385022891e-07 -0.05 -0.014912246259012996" rpy="0 0 0"/>
     <mass value="12.646385127140846"/>
     <inertia ixx="0.752015" iyy="0.005192" izz="0.755318" ixy="0.0" iyz="0.0" ixz="-0.0"/>
   </inertial>
   <visual>
-    <origin xyz="0.44955 -0.05752 -0.376" rpy="0 0 0"/>
+    <origin xyz="0.44955 -0.10752 -0.376" rpy="0 0 0"/>
     <geometry>
       <mesh filename="package://4ws_backstepping/meshes/v1_rear_1.stl" scale="0.001 0.001 0.001"/>
@@ -72,5 +72,5 @@
   </visual>
   <collision>
-    <origin xyz="0.44955 -0.05752 -0.376" rpy="0 0 0"/>
+    <origin xyz="0.44955 -0.10752 -0.376" rpy="0 0 0"/>
     <geometry>
       <mesh filename="package://4ws_backstepping/meshes/v1_rear_1.stl" scale="0.001 0.001 0.001"/>
@@ -80,10 +80,10 @@
 <link name="v1_front_1">
   <inertial>
-    <origin xyz="2.5142643794717756e-07 2.540691661362393e-07 -0.014912246259013162" rpy="0 0 0"/>
+    <origin xyz="2.5142643794717756e-07 -0.05 -0.014912246259013162" rpy="0 0 0"/>
     <mass value="12.64638512714101"/>
     <inertia ixx="0.752015" iyy="0.005192" izz="0.755318" ixy="-0.0" iyz="0.0" ixz="-0.0"/>
   </inertial>
   <visual>
-    <origin xyz="-0.45045 -0.05752 -0.376" rpy="0 0 0"/>
+    <origin xyz="-0.45045 -0.10752 -0.376" rpy="0 0 0"/>
     <geometry>
       <mesh filename="package://4ws_backstepping/meshes/v1_front_1.stl" scale="0.001 0.001 0.001"/>
@@ -92,5 +92,5 @@
   </visual>
   <collision>
-    <origin xyz="-0.45045 -0.05752 -0.376" rpy="0 0 0"/>
+    <origin xyz="-0.45045 -0.10752 -0.376" rpy="0 0 0"/>
     <geometry>
       <mesh filename="package://4ws_backstepping/meshes/v1_front_1.stl" scale="0.001 0.001 0.001"/>
@@ -100,10 +100,10 @@
 <link name="new_hinge_1">
   <inertial>
-    <origin xyz="-6.714468377522209e-05 2.5406917214532143e-07 -0.11523004751915897" rpy="0 0 0"/>
+    <origin xyz="-6.714468377522209e-05 -0.05 -0.11523004751915897" rpy="0 0 0"/>
     <mass value="4.884144703315957"/>
     <inertia ixx="0.039519" iyy="0.032652" izz="0.021551" ixy="0.0" iyz="0.0" ixz="-3e-05"/>
   </inertial>
   <visual>
-    <origin xyz="-0.45045 0.34248 -0.356" rpy="0 0 0"/>
+    <origin xyz="-0.45045 0.29248 -0.356" rpy="0 0 0"/>
     <geometry>
       <mesh filename="package://4ws_backstepping/meshes/new_hinge_1.stl" scale="0.001 0.001 0.001"/>
@@ -112,5 +112,5 @@
   </visual>
   <collision>
-    <origin xyz="-0.45045 0.34248 -0.356" rpy="0 0 0"/>
+    <origin xyz="-0.45045 0.29248 -0.356" rpy="0 0 0"/>
     <geometry>
       <mesh filename="package://4ws_backstepping/meshes/new_hinge_1.stl" scale="0.001 0.001 0.001"/>
@@ -120,10 +120,10 @@
 <link name="new_hinge_3">
   <inertial>
-    <origin xyz="-6.714468377522209e-05 2.5406917258941064e-07 -0.11523004751915977" rpy="0 0 0"/>
+    <origin xyz="-6.714468377522209e-05 -0.05 -0.11523004751915977" rpy="0 0 0"/>
     <mass value="4.884144703315957"/>
     <inertia ixx="0.039519" iyy="0.032652" izz="0.021551" ixy="-0.0" iyz="0.0" ixz="-3e-05"/>
   </inertial>
   <visual>
-    <origin xyz="-0.45045 -0.45752 -0.356" rpy="0 0 0"/>
+    <origin xyz="-0.45045 -0.50752 -0.356" rpy="0 0 0"/>
     <geometry>
       <mesh filename="package://4ws_backstepping/meshes/new_hinge_3.stl" scale="0.001 0.001 0.001"/>
@@ -132,5 +132,5 @@
   </visual>
   <collision>
-    <origin xyz="-0.45045 -0.45752 -0.356" rpy="0 0 0"/>
+    <origin xyz="-0.45045 -0.50752 -0.356" rpy="0 0 0"/>
     <geometry>
       <mesh filename="package://4ws_backstepping/meshes/new_hinge_3.stl" scale="0.001 0.001 0.001"/>
@@ -140,10 +140,10 @@
 <link name="new_hinge_2">
   <inertial>
-    <origin xyz="-6.714468377322369e-05 2.540692444763515e-07 -0.1152300475191588" rpy="0 0 0"/>
+    <origin xyz="-6.714468377322369e-05 -0.05 -0.1152300475191588" rpy="0 0 0"/>
     <mass value="4.884144703315957"/>
     <inertia ixx="0.039519" iyy="0.032652" izz="0.021551" ixy="0.0" iyz="0.0" ixz="-3e-05"/>
   </inertial>
   <visual>
-    <origin xyz="0.44955 0.34248 -0.356" rpy="0 0 0"/>
+    <origin xyz="0.44955 0.29248 -0.356" rpy="0 0 0"/>
     <geometry>
       <mesh filename="package://4ws_backstepping/meshes/new_hinge_2.stl" scale="0.001 0.001 0.001"/>
@@ -152,5 +152,5 @@
   </visual>
   <collision>
-    <origin xyz="0.44955 0.34248 -0.356" rpy="0 0 0"/>
+    <origin xyz="0.44955 0.29248 -0.356" rpy="0 0 0"/>
     <geometry>
       <mesh filename="package://4ws_backstepping/meshes/new_hinge_2.stl" scale="0.001 0.001 0.001"/>
@@ -160,10 +160,10 @@
 <link name="new_hinge_4">
   <inertial>
-    <origin xyz="-6.714468377405636e-05 2.5406924475390724e-07 -0.11523004751915963" rpy="0 0 0"/>
+    <origin xyz="-6.714468377405636e-05 -0.05 -0.11523004751915963" rpy="0 0 0"/>
     <mass value="4.884144703315957"/>
     <inertia ixx="0.039519" iyy="0.032652" izz="0.021551" ixy="0.0" iyz="0.0" ixz="-3e-05"/>
   </inertial>
   <visual>
-    <origin xyz="0.44955 -0.45752 -0.356" rpy="0 0 0"/>
+    <origin xyz="0.44955 -0.50752 -0.356" rpy="0 0 0"/>
     <geometry>
       <mesh filename="package://4ws_backstepping/meshes/new_hinge_4.stl" scale="0.001 0.001 0.001"/>
@@ -172,5 +172,5 @@
   </visual>
   <collision>
-    <origin xyz="0.44955 -0.45752 -0.356" rpy="0 0 0"/>
+    <origin xyz="0.44955 -0.50752 -0.356" rpy="0 0 0"/>
     <geometry>
       <mesh filename="package://4ws_backstepping/meshes/new_hinge_4.stl" scale="0.001 0.001 0.001"/>
@@ -181,10 +181,10 @@
 <link name="new_wheel_1">
   <inertial>
-    <origin xyz="3.1709373395083507e-05 2.540692010666312e-07 0.00021681028363659816" rpy="0 0 0"/>
+    <origin xyz="3.1709373395083507e-05 -0.05 0.00021681028363659816" rpy="0 0 0"/>
     <mass value="4.639715839283939"/>
     <inertia ixx="0.029034" iyy="0.053334" izz="0.029034" ixy="-0.0" iyz="0.0" ixz="0.0"/>
   </inertial>
   <visual>
-    <origin xyz="-0.450031 0.34248 -0.150215" rpy="0 0 0"/>
+    <origin xyz="-0.450031 0.29248 -0.150215" rpy="0 0 0"/>
     <geometry>
       <mesh filename="package://4ws_backstepping/meshes/new_wheel_1.stl" scale="0.001 0.001 0.001"/>
@@ -218,10 +218,10 @@
 <link name="new_wheel_2">
   <inertial>
-    <origin xyz="3.1709373397914575e-05 2.5406927345317243e-07 0.00021681028363673693" rpy="0 0 0"/>
+    <origin xyz="3.1709373397914575e-05 -0.05 0.00021681028363673693" rpy="0 0 0"/>
     <mass value="4.639715839283939"/>
     <inertia ixx="0.029034" iyy="0.053334" izz="0.029034" ixy="0.0" iyz="0.0" ixz="0.0"/>
   </inertial>
   <visual>
-    <origin xyz="0.449969 0.34248 -0.150215" rpy="0 0 0"/>
+    <origin xyz="0.449969 0.29248 -0.150215" rpy="0 0 0"/>
     <geometry>
       <mesh filename="package://4ws_backstepping/meshes/new_wheel_2.stl" scale="0.001 0.001 0.001"/>
@@ -230,5 +230,5 @@
   </visual>
   <collision>
-    <!-- <origin xyz="0.449969 0.34248 -0.150215" rpy="0 0 0"/>
+    <!-- <origin xyz="0.449969 0.29248 -0.150215" rpy="0 0 0"/>
     <geometry>
       <mesh filename="package://4ws_backstepping/meshes/new_wheel_2.stl" scale="0.001 0.001 0.001"/>
@@ -259,10 +259,10 @@
 <link name="new_wheel_3">
   <inertial>
-    <origin xyz="3.1709373395083507e-05 2.540692015662316e-07 0.00021681028363579324" rpy="0 0 0"/>
+    <origin xyz="3.1709373395083507e-05 -0.05 0.00021681028363579324" rpy="0 0 0"/>
     <mass value="4.639715839283939"/>
     <inertia ixx="0.029034" iyy="0.053334" izz="0.029034" ixy="0.0" iyz="0.0" ixz="0.0"/>
   </inertial>
   <visual>
-    <origin xyz="-0.450031 -0.45752 -0.150215" rpy="0 0 0"/>
+    <origin xyz="-0.450031 -0.50752 -0.150215" rpy="0 0 0"/>
     <geometry>
       <mesh filename="package://4ws_backstepping/meshes/new_wheel_3.stl" scale="0.001 0.001 0.001"/>
@@ -271,5 +271,5 @@
   </visual>
   <collision>
-    <!-- <origin xyz="-0.450031 -0.45752 -0.150215" rpy="0 0 0"/>
+    <!-- <origin xyz="-0.450031 -0.50752 -0.150215" rpy="0 0 0"/>
     <geometry>
       <mesh filename="package://4ws_backstepping/meshes/new_wheel_3.stl" scale="0.001 0.001 0.001"/>
@@ -300,10 +300,10 @@
 <link name="new_wheel_4">
   <inertial>
-    <origin xyz="3.170937339708191e-05 2.540692737307282e-07 0.00021681028363593202" rpy="0 0 0"/>
+    <origin xyz="3.170937339708191e-05 -0.05 0.00021681028363593202" rpy="0 0 0"/>
     <mass value="4.639715839283939"/>
     <inertia ixx="0.029034" iyy="0.053334" izz="0.029034" ixy="0.0" iyz="0.0" ixz="0.0"/>
   </inertial>
   <visual>
-    <origin xyz="0.449969 -0.45752 -0.150215" rpy="0 0 0"/>
+    <origin xyz="0.449969 -0.50752 -0.150215" rpy="0 0 0"/>
     <geometry>
       <mesh filename="package://4ws_backstepping/meshes/new_wheel_4.stl" scale="0.001 0.001 0.001"/>
@@ -312,5 +312,5 @@
   </visual>
   <collision>
-    <!-- <origin xyz="0.449969 -0.45752 -0.150215" rpy="0 0 0"/>
+    <!-- <origin xyz="0.449969 -0.50752 -0.150215" rpy="0 0 0"/>
     <geometry>
       <mesh filename="package://4ws_backstepping/meshes/new_wheel_4.stl" scale="0.001 0.001 0.001"/>
