Commit message: 少しタイヤの空転が見られたが一旦登った

File: urdf/vehicle_4ws_real_hill.xacro (robot description, xacro)
@@ -8,22 +8,31 @@
 <xacro:property name="vehicle_body_mass" value="100" />
 <xacro:property name="vehicle_inertia_coef" value="${vehicle_body_mass/fusion_vehicle_body_mass}" />
+<!-- 車輪のmass -->
+<xacro:property name="fusion_wheel_mass" value="4.639715839283939" />
+<xacro:property name="vehicle_wheel_mass" value="12" />
+<xacro:property name="wheel_inertia_coef" value="${vehicle_wheel_mass/fusion_wheel_mass}" />
 <xacro:property name="wheel_mass" value="4.639715839283939" />
+<!-- ステアリングのmass -->
+<xacro:property name="fusion_hinge_mass" value="4.639715839283939" />
+<xacro:property name="vehicle_hinge_mass" value="12" />
+<xacro:property name="hinge_inertia_coef" value="${vehicle_hinge_mass/fusion_hinge_mass}" />
+<xacro:property name="hinge_mass" value="4.639715839283939" />
 <!-- frontは受動車輪なので低めに設定 -->
 <xacro:property name="front_wheel_joint_damping" value="1.0"/>
-<xacro:property name="front_wheel_joint_mu" value="0.1" />
+<xacro:property name="front_wheel_joint_mu" value="0.01" />
 <xacro:property name="front_wheel_joint_friction" value="${front_wheel_joint_mu* gravitational_acceleration * wheel_mass  }" />
-<xacro:property name="front_steering_damping" value="3.0" />
-<xacro:property name="front_steering_mu" value="0.01" />
+<xacro:property name="front_steering_damping" value="2.0" />
+<xacro:property name="front_steering_mu" value="0.1" />
 <xacro:property name="front_steering_friction" value="${front_steering_mu * gravitational_acceleration * 0.25*vehicle_body_mass}" />
 <!-- rearは駆動輪なので、入力以外で動かないように設定 -->
 <xacro:property name="rear_wheel_joint_damping" value="1.0"/>
-<xacro:property name="rear_wheel_joint_mu" value="0.1" />
+<xacro:property name="rear_wheel_joint_mu" value="0.01" />
 <xacro:property name="rear_wheel_joint_friction" value="${rear_wheel_joint_mu* gravitational_acceleration * wheel_mass }" />
-<xacro:property name="rear_steering_damping" value="3.0" />
-<xacro:property name="rear_steering_mu" value="0.01" />
+<xacro:property name="rear_steering_damping" value="2.0" />
+<xacro:property name="rear_steering_mu" value="0.1" />
 <xacro:property name="rear_steering_friction" value="${rear_steering_mu * gravitational_acceleration * 0.25*vehicle_body_mass}" />
 <!-- wheelの接地面の摩擦などを定義 -->
-<xacro:property name="wheel_surface_mu1" value="2.0"/>
-<xacro:property name="wheel_surface_mu2" value="2.0" />
+<xacro:property name="wheel_surface_mu1" value="1.2"/>
+<xacro:property name="wheel_surface_mu2" value="1.2" />
 <xacro:property name="wheel_kp" value="5e4" />
 <xacro:property name="wheel_kd" value="1.0" />
@@ -60,5 +69,5 @@
 <link name="v1_rear_1">
   <inertial>
-    <origin xyz="2.514264385022891e-07 -0.05 -0.014912246259012996" rpy="0 0 0"/>
+    <origin xyz="2.514264385022891e-07 2.540692383215526e-07 -0.014912246259012996" rpy="0 0 0"/>
     <mass value="12.646385127140846"/>
     <inertia ixx="0.752015" iyy="0.005192" izz="0.755318" ixy="0.0" iyz="0.0" ixz="-0.0"/>
@@ -80,5 +89,5 @@
 <link name="v1_front_1">
   <inertial>
-    <origin xyz="2.5142643794717756e-07 -0.05 -0.014912246259013162" rpy="0 0 0"/>
+    <origin xyz="2.5142643794717756e-07 2.540691661362393e-07 -0.014912246259013162" rpy="0 0 0"/>
     <mass value="12.64638512714101"/>
     <inertia ixx="0.752015" iyy="0.005192" izz="0.755318" ixy="-0.0" iyz="0.0" ixz="-0.0"/>
@@ -100,10 +109,10 @@
 <link name="new_hinge_1">
   <inertial>
-    <origin xyz="-6.714468377522209e-05 -0.05 -0.11523004751915897" rpy="0 0 0"/>
-    <mass value="4.884144703315957"/>
-    <inertia ixx="0.039519" iyy="0.032652" izz="0.021551" ixy="0.0" iyz="0.0" ixz="-3e-05"/>
-  </inertial>
-  <visual>
-    <origin xyz="-0.45045 0.29248 -0.356" rpy="0 0 0"/>
+    <origin xyz="-6.714468377522209e-05 2.5406917214532143e-07 -0.11523004751915897" rpy="0 0 0"/>
+    <mass value="${vehicle_hinge_mass}"/>
+    <inertia ixx="${hinge_inertia_coef*0.039519}" iyy="${hinge_inertia_coef*0.032652}" izz="${hinge_inertia_coef*0.021551}" ixy="0.0" iyz="0.0" ixz="-3e-05"/>
+  </inertial>
+  <visual>
+    <origin xyz="-0.45045 0.34248 -0.356" rpy="0 0 0"/>
     <geometry>
       <mesh filename="package://4ws_backstepping/meshes/new_hinge_1.stl" scale="0.001 0.001 0.001"/>
@@ -112,5 +121,5 @@
   </visual>
   <collision>
-    <origin xyz="-0.45045 0.29248 -0.356" rpy="0 0 0"/>
+    <origin xyz="-0.45045 0.34248 -0.356" rpy="0 0 0"/>
     <geometry>
       <mesh filename="package://4ws_backstepping/meshes/new_hinge_1.stl" scale="0.001 0.001 0.001"/>
@@ -120,10 +129,10 @@
 <link name="new_hinge_3">
   <inertial>
-    <origin xyz="-6.714468377522209e-05 -0.05 -0.11523004751915977" rpy="0 0 0"/>
-    <mass value="4.884144703315957"/>
-    <inertia ixx="0.039519" iyy="0.032652" izz="0.021551" ixy="-0.0" iyz="0.0" ixz="-3e-05"/>
-  </inertial>
-  <visual>
-    <origin xyz="-0.45045 -0.50752 -0.356" rpy="0 0 0"/>
+    <origin xyz="-6.714468377522209e-05 2.5406917258941064e-07 -0.11523004751915977" rpy="0 0 0"/>
+    <mass value="${vehicle_hinge_mass}"/>
+    <inertia ixx="${hinge_inertia_coef*0.039519}" iyy="${hinge_inertia_coef*0.032652}" izz="${hinge_inertia_coef*0.021551}" ixy="-0.0" iyz="0.0" ixz="-3e-05"/>
+  </inertial>
+  <visual>
+    <origin xyz="-0.45045 -0.45752 -0.356" rpy="0 0 0"/>
     <geometry>
       <mesh filename="package://4ws_backstepping/meshes/new_hinge_3.stl" scale="0.001 0.001 0.001"/>
@@ -132,5 +141,5 @@
   </visual>
   <collision>
-    <origin xyz="-0.45045 -0.50752 -0.356" rpy="0 0 0"/>
+    <origin xyz="-0.45045 -0.45752 -0.356" rpy="0 0 0"/>
     <geometry>
       <mesh filename="package://4ws_backstepping/meshes/new_hinge_3.stl" scale="0.001 0.001 0.001"/>
@@ -140,10 +149,10 @@
 <link name="new_hinge_2">
   <inertial>
-    <origin xyz="-6.714468377322369e-05 -0.05 -0.1152300475191588" rpy="0 0 0"/>
-    <mass value="4.884144703315957"/>
-    <inertia ixx="0.039519" iyy="0.032652" izz="0.021551" ixy="0.0" iyz="0.0" ixz="-3e-05"/>
-  </inertial>
-  <visual>
-    <origin xyz="0.44955 0.29248 -0.356" rpy="0 0 0"/>
+    <origin xyz="-6.714468377322369e-05 2.540692444763515e-07 -0.1152300475191588" rpy="0 0 0"/>
+    <mass value="${vehicle_hinge_mass}"/>
+    <inertia ixx="${hinge_inertia_coef*0.039519}" iyy="${hinge_inertia_coef*0.032652}" izz="${hinge_inertia_coef*0.021551}" ixy="0.0" iyz="0.0" ixz="-3e-05"/>
+  </inertial>
+  <visual>
+    <origin xyz="0.44955 0.34248 -0.356" rpy="0 0 0"/>
     <geometry>
       <mesh filename="package://4ws_backstepping/meshes/new_hinge_2.stl" scale="0.001 0.001 0.001"/>
@@ -152,5 +161,5 @@
   </visual>
   <collision>
-    <origin xyz="0.44955 0.29248 -0.356" rpy="0 0 0"/>
+    <origin xyz="0.44955 0.34248 -0.356" rpy="0 0 0"/>
     <geometry>
       <mesh filename="package://4ws_backstepping/meshes/new_hinge_2.stl" scale="0.001 0.001 0.001"/>
@@ -160,10 +169,10 @@
 <link name="new_hinge_4">
   <inertial>
-    <origin xyz="-6.714468377405636e-05 -0.05 -0.11523004751915963" rpy="0 0 0"/>
-    <mass value="4.884144703315957"/>
-    <inertia ixx="0.039519" iyy="0.032652" izz="0.021551" ixy="0.0" iyz="0.0" ixz="-3e-05"/>
-  </inertial>
-  <visual>
-    <origin xyz="0.44955 -0.50752 -0.356" rpy="0 0 0"/>
+    <origin xyz="-6.714468377405636e-05 2.5406924475390724e-07 -0.11523004751915963" rpy="0 0 0"/>
+    <mass value="${vehicle_hinge_mass}"/>
+    <inertia ixx="${hinge_inertia_coef*0.039519}" iyy="${hinge_inertia_coef*0.032652}" izz="${hinge_inertia_coef*0.021551}" ixy="0.0" iyz="0.0" ixz="-3e-05"/>
+  </inertial>
+  <visual>
+    <origin xyz="0.44955 -0.45752 -0.356" rpy="0 0 0"/>
     <geometry>
       <mesh filename="package://4ws_backstepping/meshes/new_hinge_4.stl" scale="0.001 0.001 0.001"/>
@@ -172,5 +181,5 @@
   </visual>
   <collision>
-    <origin xyz="0.44955 -0.50752 -0.356" rpy="0 0 0"/>
+    <origin xyz="0.44955 -0.45752 -0.356" rpy="0 0 0"/>
     <geometry>
       <mesh filename="package://4ws_backstepping/meshes/new_hinge_4.stl" scale="0.001 0.001 0.001"/>
@@ -181,10 +190,10 @@
 <link name="new_wheel_1">
   <inertial>
-    <origin xyz="3.1709373395083507e-05 -0.05 0.00021681028363659816" rpy="0 0 0"/>
-    <mass value="4.639715839283939"/>
-    <inertia ixx="0.029034" iyy="0.053334" izz="0.029034" ixy="-0.0" iyz="0.0" ixz="0.0"/>
-  </inertial>
-  <visual>
-    <origin xyz="-0.450031 0.29248 -0.150215" rpy="0 0 0"/>
+    <origin xyz="3.1709373395083507e-05 2.540692010666312e-07 0.00021681028363659816" rpy="0 0 0"/>
+    <mass value="${vehicle_wheel_mass}"/>
+    <inertia ixx="${wheel_inertia_coef*0.029034}" iyy="${wheel_inertia_coef*0.053334}" izz="${wheel_inertia_coef*0.029034}" ixy="-0.0" iyz="0.0" ixz="0.0"/>
+  </inertial>
+  <visual>
+    <origin xyz="-0.450031 0.34248 -0.150215" rpy="0 0 0"/>
     <geometry>
       <mesh filename="package://4ws_backstepping/meshes/new_wheel_1.stl" scale="0.001 0.001 0.001"/>
@@ -218,10 +227,10 @@
 <link name="new_wheel_2">
   <inertial>
-    <origin xyz="3.1709373397914575e-05 -0.05 0.00021681028363673693" rpy="0 0 0"/>
-    <mass value="4.639715839283939"/>
-    <inertia ixx="0.029034" iyy="0.053334" izz="0.029034" ixy="0.0" iyz="0.0" ixz="0.0"/>
-  </inertial>
-  <visual>
-    <origin xyz="0.449969 0.29248 -0.150215" rpy="0 0 0"/>
+    <origin xyz="3.1709373397914575e-05 2.5406927345317243e-07 0.00021681028363673693" rpy="0 0 0"/>
+    <mass value="${vehicle_wheel_mass}"/>
+    <inertia ixx="${wheel_inertia_coef*0.029034}" iyy="${wheel_inertia_coef*0.053334}" izz="${wheel_inertia_coef*0.029034}"  ixy="0.0" iyz="0.0" ixz="0.0"/>
+  </inertial>
+  <visual>
+    <origin xyz="0.449969 0.34248 -0.150215" rpy="0 0 0"/>
     <geometry>
       <mesh filename="package://4ws_backstepping/meshes/new_wheel_2.stl" scale="0.001 0.001 0.001"/>
@@ -259,10 +268,10 @@
 <link name="new_wheel_3">
   <inertial>
-    <origin xyz="3.1709373395083507e-05 -0.05 0.00021681028363579324" rpy="0 0 0"/>
-    <mass value="4.639715839283939"/>
-    <inertia ixx="0.029034" iyy="0.053334" izz="0.029034" ixy="0.0" iyz="0.0" ixz="0.0"/>
-  </inertial>
-  <visual>
-    <origin xyz="-0.450031 -0.50752 -0.150215" rpy="0 0 0"/>
+    <origin xyz="3.1709373395083507e-05 2.540692015662316e-07 0.00021681028363579324" rpy="0 0 0"/>
+    <mass value="${vehicle_wheel_mass}"/>
+    <inertia ixx="${wheel_inertia_coef*0.029034}" iyy="${wheel_inertia_coef*0.053334}" izz="${wheel_inertia_coef*0.029034}"  ixy="0.0" iyz="0.0" ixz="0.0"/>
+  </inertial>
+  <visual>
+    <origin xyz="-0.450031 -0.45752 -0.150215" rpy="0 0 0"/>
     <geometry>
       <mesh filename="package://4ws_backstepping/meshes/new_wheel_3.stl" scale="0.001 0.001 0.001"/>
@@ -300,10 +309,10 @@
 <link name="new_wheel_4">
   <inertial>
-    <origin xyz="3.170937339708191e-05 -0.05 0.00021681028363593202" rpy="0 0 0"/>
-    <mass value="4.639715839283939"/>
-    <inertia ixx="0.029034" iyy="0.053334" izz="0.029034" ixy="0.0" iyz="0.0" ixz="0.0"/>
-  </inertial>
-  <visual>
-    <origin xyz="0.449969 -0.50752 -0.150215" rpy="0 0 0"/>
+    <origin xyz="3.170937339708191e-05 2.540692737307282e-07 0.00021681028363593202" rpy="0 0 0"/>
+    <mass value="${vehicle_wheel_mass}"/>
+    <inertia ixx="${wheel_inertia_coef*0.029034}" iyy="${wheel_inertia_coef*0.053334}" izz="${wheel_inertia_coef*0.029034}"  ixy="0.0" iyz="0.0" ixz="0.0"/>
+  </inertial>
+  <visual>
+    <origin xyz="0.449969 -0.45752 -0.150215" rpy="0 0 0"/>
     <geometry>
       <mesh filename="package://4ws_backstepping/meshes/new_wheel_4.stl" scale="0.001 0.001 0.001"/>
@@ -340,5 +349,5 @@
 </link>
 <joint name="body" type="fixed">
-  <origin xyz="0 -0.05 0.376" rpy="0 0 0"/>
+  <origin xyz="0 0 0.376" rpy="0 0 0"/>
   <parent link="base_link"/>
   <child link="body_link"/>
@@ -355,5 +364,5 @@
 </joint>
 <joint name="front_right_steering" type="revolute">
-  <origin xyz="0.0 -0.4 -0.02" rpy="0 0 0"/>
+  <origin xyz="0.0 -0.45 -0.02" rpy="0 0 0"/>
   <parent link="v1_front_1"/>
   <child link="new_hinge_1"/>
@@ -379,5 +388,5 @@
 </joint>
 <joint name="front_left_steering" type="revolute">
-  <origin xyz="0.0 0.4 -0.02" rpy="0 0 0"/>
+  <origin xyz="0.0 0.35 -0.02" rpy="0 0 0"/>
   <parent link="v1_front_1"/>
   <child link="new_hinge_3"/>
@@ -404,5 +413,5 @@
 <!-- 後輪右ステア -->
 <joint name="rear_right_steering" type="revolute">
-  <origin xyz="0.0 -0.4 -0.02" rpy="0 0 0"/>
+  <origin xyz="0.0 -0.45 -0.02" rpy="0 0 0"/>
   <parent link="v1_rear_1"/>
   <child  link="new_hinge_2"/>
@@ -416,5 +425,5 @@
 <!-- 後輪左ステア -->
 <joint name="rear_left_steering" type="revolute">
-  <origin xyz="0.0 0.4 -0.02" rpy="0 0 0"/>
+  <origin xyz="0.0 0.35 -0.02" rpy="0 0 0"/>
   <parent link="v1_rear_1"/>
   <child  link="new_hinge_4"/>

Commit message: 坂道用ゲイン変更

File: urdf/vehicle_4ws_real_hill.xacro (robot description, xacro)
@@ -22,5 +22,5 @@
 <xacro:property name="front_wheel_joint_mu" value="0.01" />
 <xacro:property name="front_wheel_joint_friction" value="${front_wheel_joint_mu* gravitational_acceleration * wheel_mass  }" />
-<xacro:property name="front_steering_damping" value="2.0" />
+<xacro:property name="front_steering_damping" value="1.0" />
 <xacro:property name="front_steering_mu" value="0.1" />
 <xacro:property name="front_steering_friction" value="${front_steering_mu * gravitational_acceleration * 0.25*vehicle_body_mass}" />
@@ -29,5 +29,5 @@
 <xacro:property name="rear_wheel_joint_mu" value="0.01" />
 <xacro:property name="rear_wheel_joint_friction" value="${rear_wheel_joint_mu* gravitational_acceleration * wheel_mass }" />
-<xacro:property name="rear_steering_damping" value="2.0" />
+<xacro:property name="rear_steering_damping" value="1.0" />
 <xacro:property name="rear_steering_mu" value="0.1" />
 <xacro:property name="rear_steering_friction" value="${rear_steering_mu * gravitational_acceleration * 0.25*vehicle_body_mass}" />
@@ -35,8 +35,8 @@
 <xacro:property name="wheel_surface_mu1" value="1.2"/>
 <xacro:property name="wheel_surface_mu2" value="1.2" />
-<xacro:property name="wheel_kp" value="5e4" />
-<xacro:property name="wheel_kd" value="1.0" />
-<xacro:property name="wheel_minDepth" value="0.01" />
-<xacro:property name="wheel_maxVel" value="1.0" />
+<xacro:property name="wheel_kp" value="8e4" />
+<xacro:property name="wheel_kd" value="50" />
+<xacro:property name="wheel_minDepth" value="0.005" />
+<xacro:property name="wheel_maxVel" value="2.0" />
 <!-- rotationは共通 -->
 <xacro:property name="rotational_joint_damping" value="0.01" />

Commit message: Consideration of load on hill

File: urdf/vehicle_4ws_real_hill.xacro (robot description, xacro)
@@ -10,10 +10,10 @@
 <!-- 車輪のmass -->
 <xacro:property name="fusion_wheel_mass" value="4.639715839283939" />
-<xacro:property name="vehicle_wheel_mass" value="12" />
+<xacro:property name="vehicle_wheel_mass" value="8" />
 <xacro:property name="wheel_inertia_coef" value="${vehicle_wheel_mass/fusion_wheel_mass}" />
 <xacro:property name="wheel_mass" value="4.639715839283939" />
 <!-- ステアリングのmass -->
 <xacro:property name="fusion_hinge_mass" value="4.639715839283939" />
-<xacro:property name="vehicle_hinge_mass" value="8" />
+<xacro:property name="vehicle_hinge_mass" value="12" />
 <xacro:property name="hinge_inertia_coef" value="${vehicle_hinge_mass/fusion_hinge_mass}" />
 <xacro:property name="hinge_mass" value="4.639715839283939" />
@@ -21,5 +21,5 @@
 <xacro:property name="front_wheel_joint_damping" value="1.0"/>
 <xacro:property name="front_wheel_joint_mu" value="0.01" />
-<xacro:property name="front_wheel_joint_friction" value="${front_wheel_joint_mu* gravitational_acceleration * wheel_mass  }" />
+<xacro:property name="front_wheel_joint_friction" value="${front_wheel_joint_mu* gravitational_acceleration * vehicle_wheel_mass  }" />
 <xacro:property name="front_steering_damping" value="1.0" />
 <xacro:property name="front_steering_mu" value="0.1" />
@@ -28,5 +28,5 @@
 <xacro:property name="rear_wheel_joint_damping" value="1.0"/>
 <xacro:property name="rear_wheel_joint_mu" value="0.01" />
-<xacro:property name="rear_wheel_joint_friction" value="${rear_wheel_joint_mu* gravitational_acceleration * wheel_mass }" />
+<xacro:property name="rear_wheel_joint_friction" value="${rear_wheel_joint_mu* gravitational_acceleration * vehicle_wheel_mass }" />
 <xacro:property name="rear_steering_damping" value="1.0" />
 <xacro:property name="rear_steering_mu" value="0.1" />

Commit message: hill完走_20250826

File: urdf/vehicle_4ws_real_hill.xacro (robot description, xacro)
@@ -33,6 +33,6 @@
 <xacro:property name="rear_steering_friction" value="${rear_steering_mu * gravitational_acceleration * 0.25*vehicle_body_mass}" />
 <!-- wheelの接地面の摩擦などを定義 -->
-<xacro:property name="wheel_surface_mu1" value="1.2"/>
-<xacro:property name="wheel_surface_mu2" value="1.2" />
+<xacro:property name="wheel_surface_mu1" value="0.8"/>
+<xacro:property name="wheel_surface_mu2" value="0.8" />
 <xacro:property name="wheel_kp" value="8e4" />
 <xacro:property name="wheel_kd" value="50" />

Commit message: muを0.6に変更

File: urdf/vehicle_4ws_real_hill.xacro (robot description, xacro)
@@ -33,6 +33,6 @@
 <xacro:property name="rear_steering_friction" value="${rear_steering_mu * gravitational_acceleration * 0.25*vehicle_body_mass}" />
 <!-- wheelの接地面の摩擦などを定義 -->
-<xacro:property name="wheel_surface_mu1" value="0.8"/>
-<xacro:property name="wheel_surface_mu2" value="0.8" />
+<xacro:property name="wheel_surface_mu1" value="0.6"/>
+<xacro:property name="wheel_surface_mu2" value="0.6" />
 <xacro:property name="wheel_kp" value="8e4" />
 <xacro:property name="wheel_kd" value="50" />

Commit message: muに差異をつける

File: urdf/vehicle_4ws_real_hill.xacro (robot description, xacro)
@@ -33,8 +33,8 @@
 <xacro:property name="rear_steering_friction" value="${rear_steering_mu * gravitational_acceleration * 0.25*vehicle_body_mass}" />
 <!-- wheelの接地面の摩擦などを定義 -->
-<xacro:property name="wheel_surface_mu1" value="0.6"/>
+<xacro:property name="wheel_surface_mu1" value="0.8"/>
 <xacro:property name="wheel_surface_mu2" value="0.6" />
 <xacro:property name="wheel_kp" value="8e4" />
-<xacro:property name="wheel_kd" value="50" />
+<xacro:property name="wheel_kd" value="300" />
 <xacro:property name="wheel_minDepth" value="0.005" />
 <xacro:property name="wheel_maxVel" value="2.0" />
